Commit message: Feature 1: spawn few parts on a field with detouchable joints. TODO: attach and detach only connected voxel/part

File: ros2_ws/src/srrs_sim/urdf/temp_robot.urdf (robot description, URDF)
Before this commit: robot rel_robot, 21 links, 20 joints
Links:
- removed link camera_link
- removed link camera_link_optical
- added link camera1; visual box size=0.01 0.01 0.01
- added link camera1_optical
- added link camera2; visual box size=0.01 0.01 0.01
- added link camera2_optical
- link contact1: geometry collision cylinder length=0.002 radius=0.05; visual cylinder length=0.002 radius=0.05
- link contact2: geometry collision cylinder length=0.002 radius=0.05; visual cylinder length=0.002 radius=0.05
Joints:
- removed joint camera_joint
- removed joint camera_optical_joint
- added joint camera1_joint: type fixed, parent block0_fix, child camera1, origin xyz=0 0 0 rpy=0 1.5707963267948966 0
- added joint camera1_optical_joint: type fixed, parent camera1, child camera1_optical, origin xyz=0 0 0 rpy=-1.5707963267948966 0 -1.5707963267948966
- added joint camera2_joint: type fixed, parent block14fix, child camera2, origin xyz=0 0 0.134 rpy=0 -1.5707963267948966 0
- added joint camera2_optical_joint: type fixed, parent camera2, child camera2_optical, origin xyz=0 0 0 rpy=-1.5707963267948966 0 -1.5707963267948966
- joint contact2_joint: origin xyz=0 0 0.137 -> xyz=0 0 0.134
