Commit message: add pose publish node

File: ros2_ws/src/srrs_sim/urdf/part.xacro (robot description, xacro)
@@ -1,49 +1,68 @@
 <?xml version="1.0" ?>
 <robot name="part" xmlns:xacro="http://www.ros.org/wiki/xacro">
-<xacro:arg name="part_num" default="0"/>
-  <link name="part">
-    <visual>
-      <geometry>
-          <mesh filename="/home/lao/Documents/Masterarbeit/git/SRRS_gazebo_sim/ros2_ws/src/srrs_sim/meshes/Voxel.stl" scale="0.001 0.001 0.001"/>
-          <!-- <box size="0.1 0.1 0.1"/> -->
-      </geometry>
-    </visual>
-    <collision name="part_collision">
-        <geometry>
-        <mesh filename="/home/lao/Documents/Masterarbeit/git/SRRS_gazebo_sim/ros2_ws/src/srrs_sim/meshes/Voxel.stl" scale="0.001 0.001 0.001"/>
-          <!-- <box size="0.1 0.1 0.1"/> -->
-        </geometry>
-    </collision>
-    <inertial>
-      <mass value="0.1"/>
-      <inertia ixx="1.0" ixy="0.0" ixz="0.0" iyy="1.0" iyz="0.0" izz="1.0"/>
-    </inertial>
-  </link>
-  <gazebo>
-    <!-- <plugin filename="gz_ros2_control-system" name="gz_ros2_control::GazeboSimROS2ControlPlugin">
+    <xacro:arg name="part_num" default="0"/>
+    <!-- <xacro:arg name="parent_model" default="0"/> -->
+    <!-- <xacro:arg name="parent_link" default="0"/> -->
+    <link name="part">
+        <visual>
+            <geometry>
+                <mesh filename="/home/lao/Documents/Masterarbeit/git/SRRS_gazebo_sim/ros2_ws/src/srrs_sim/meshes/Voxel.stl" scale="0.001 0.001 0.001"/>
+                <!-- <box size="0.1 0.1 0.1"/> -->
+            </geometry>
+        </visual>
+        <collision name="part_collision">
+            <geometry>
+                <mesh filename="/home/lao/Documents/Masterarbeit/git/SRRS_gazebo_sim/ros2_ws/src/srrs_sim/meshes/Voxel.stl" scale="0.001 0.001 0.001"/>
+                <!-- <box size="0.1 0.1 0.1"/> -->
+            </geometry>
+        </collision>
+        <inertial>
+            <mass value="0.1"/>
+            <inertia ixx="1.0" ixy="0.0" ixz="0.0" iyy="1.0" iyz="0.0" izz="1.0"/>
+        </inertial>
+    </link>
+    <gazebo>
+        <!-- <plugin filename="gz_ros2_control-system" name="gz_ros2_control::GazeboSimROS2ControlPlugin">
       <parameters>$(find srrs_sim)/config/robot_controller.yaml</parameters>
     </plugin> -->
-    <plugin
-      filename="libgz-sim8-detachable-joint-system.so"
-      name="gz::sim::systems::DetachableJoint">
-      <parent_link>part</parent_link>
-      <child_model>robot</child_model>
-      <child_link>block0_fix</child_link>
-      <attach_topic>attach_link1_obj_${xacro.arg('part_num')}</attach_topic>
-      <detach_topic>detach1_objects</detach_topic>
-      <output_topic>detachable_obj_link1_state${xacro.arg('part_num')}</output_topic>
-      <suppress_child_warning>true</suppress_child_warning>
-    </plugin>
-    <plugin
-      filename="libgz-sim8-detachable-joint-system.so"
-      name="gz::sim::systems::DetachableJoint">
-      <parent_link>part</parent_link>
-      <child_model>robot</child_model>
-      <child_link>block14fix</child_link>
-      <attach_topic>attach_link2_obj_${xacro.arg('part_num')}</attach_topic>
-      <detach_topic>detach2_objects</detach_topic>
-      <output_topic>detachable_obj_link2_state${xacro.arg('part_num')}</output_topic>
-      <suppress_child_warning>true</suppress_child_warning>
-    </plugin>
-  </gazebo>
+        <plugin
+            filename="libgz-sim8-detachable-joint-system.so"
+            name="gz::sim::systems::DetachableJoint">
+            <parent_link>part</parent_link>
+            <child_model>robot</child_model>
+            <child_link>block0_fix</child_link>
+            <attach_topic>attach_link1_obj_${xacro.arg('part_num')}</attach_topic>
+            <detach_topic>detach1_objects</detach_topic>
+            <output_topic>detachable_obj_link1_state${xacro.arg('part_num')}</output_topic>
+            <suppress_child_warning>true</suppress_child_warning>
+        </plugin>
+        <plugin
+            filename="libgz-sim8-detachable-joint-system.so"
+            name="gz::sim::systems::DetachableJoint">
+            <parent_link>part</parent_link>
+            <child_model>robot</child_model>
+            <child_link>block14fix</child_link>
+            <attach_topic>attach_link2_obj_${xacro.arg('part_num')}</attach_topic>
+            <detach_topic>detach2_objects</detach_topic>
+            <output_topic>detachable_obj_link2_state${xacro.arg('part_num')}</output_topic>
+            <suppress_child_warning>true</suppress_child_warning>
+        </plugin>
+        <!-- TODO: correct plugin to connect to previous block -->
+        <!-- <plugin -->
+        <!--     filename="libgz-sim8-detachable-joint-system.so" -->
+        <!--     name="gz::sim::systems::DetachableJoint"> -->
+        <!--     <parent_link>part</parent_link> -->
+        <!--     <child_model>${xacro.arg('parent_model')}</child_model> -->
+        <!--     <child_link>${xacro.arg('parent_link')}</child_link> -->
+        <!--     <attach_topic>attach_obj_${xacro.arg('parent_model')}</attach_topic> -->
+        <!--     <output_topic>detachable_obj_state${xacro.arg('parent_model')}</output_topic> -->
+        <!--     <suppress_child_warning>true</suppress_child_warning> -->
+        <!-- </plugin> -->
+        <plugin filename="gz-sim-pose-publisher-system" name="gz::sim::systems::PosePublisher">
+            <!-- <publish_model_pose>true</publish_model_pose> -->
+            <use_pose_vector_msg>false</use_pose_vector_msg>
+            <update_frequency>30</update_frequency>
+            <publish_nested_model_pose>true</publish_nested_model_pose>
+        </plugin>
+    </gazebo>
 </robot>
