Commit message: building robot main configuration

File: ros2_ws/src/srrs_sim/urdf/robot.xacro (robot description, xacro)
@@ -9,5 +9,5 @@
       <visual>
         <geometry>
-            <mesh filename="/home/lao/Documents/Masterarbeit/Simulation/ros2_ws/src/srrs_sim/meshes/Voxel.stl" scale="0.001 0.001 0.001"/>
+            <mesh filename="/home/lao/Documents/Masterarbeit/git/SRRS_gazebo_sim/ros2_ws/src/srrs_sim/meshes/Voxel.stl" scale="0.001 0.001 0.001"/>
         </geometry>
         <origin xyz="${origin}"/>
@@ -55,21 +55,27 @@
   <link name="world"/>
   <xacro:voxel name="block0_fix" origin="0 0 0" color="${red}"/>
+  <xacro:joint_fix name="world_to_base" parent="world" child="block0_fix"/>
   <xacro:voxel name="block1_rev" origin="0 0 0" color="${green}"/>
-  <xacro:joint_fix name="world_to_base" parent="world" child="block0_fix"/>
   <xacro:joint_revolution name="rev0_1" parent="block0_fix" child="block1_rev" axis="0 0 1" origin="0 0 ${cell_step}" rpy="0 0 0"/>
-  <xacro:voxel name="block2" origin="0 0 ${1*cell_step}" color="${blue}"/>
-  <xacro:joint_fix name="fixed1-2" parent="block1_rev" child="block2"/>
-  <xacro:voxel name="block3" origin="0 0 ${2*cell_step}" color="${blue}"/>
-  <xacro:joint_fix name="fixed2-3" parent="block2" child="block3"/>
-  <xacro:voxel name="block4_rev" origin="0 0 ${3*cell_step}" color="${green}"/>
-  <xacro:joint_fix name="fixed3-4" parent="block3" child="block4_rev"/>
-  <xacro:voxel name="block5" origin="0 ${1*cell_step} ${-0.5*cell_step}" color="${blue}"/>
-  <xacro:joint_revolution name="rev4_5" parent="block4_rev" child="block5" axis="0 1 0" origin="0 0 ${3.5*cell_step}" rpy="1.57 0 0"/>
-  <xacro:voxel name="block6" origin="0 ${1*cell_step} ${0.5*cell_step}" color="${blue}"/>
-  <xacro:joint_fix name="fixed5-6" parent="block5" child="block6"/>
-  <xacro:voxel name="block7" origin="0 ${1*cell_step} ${1.5*cell_step}" color="${blue}"/>
-  <xacro:joint_fix name="fixed6-7" parent="block6" child="block7"/>
-  <xacro:voxel name="block8" origin="0 ${1*cell_step} ${2.5*cell_step}" color="${blue}"/>
-  <xacro:joint_fix name="fixed7-8" parent="block7" child="block8"/>
+  <xacro:voxel name="block2_rev" origin="0 0 ${1*cell_step}" color="${green}"/>
+  <xacro:joint_fix name="fixed1_2" parent="block1_rev" child="block2_rev"/>
+  <xacro:voxel name="block3" origin="0 ${1*cell_step} ${-0.5*cell_step}" color="${blue}"/>
+  <xacro:joint_revolution name="rev2_3" parent="block2_rev" child="block3" axis="0 1 0" origin="0 0 ${1.5*cell_step}" rpy="1.57 0 0"/>
+  <xacro:voxel name="block4" origin="0 ${1*cell_step} ${0.5*cell_step}" color="${blue}"/>
+  <xacro:joint_fix name="fixed3_4" parent="block3" child="block4"/>
+  <xacro:voxel name="block5_rev" origin="0 ${1*cell_step} ${1.5*cell_step}" color="${green}"/>
+  <xacro:joint_fix name="fixed4_5" parent="block4" child="block5_rev"/>
+  <xacro:voxel name="block6" origin="0 ${-1*cell_step} ${-0.5*cell_step}" color="${blue}"/>
+  <xacro:joint_revolution name="rev5_6" parent="block5_rev" child="block6" axis="0 1 0" origin="0 ${1*cell_step} ${2*cell_step}" rpy="1.57 0 0"/>
+  <xacro:voxel name="block7" origin="0 ${-1*cell_step} ${0.5*cell_step}" color="${blue}"/>
+  <xacro:joint_fix name="fixed6_7" parent="block6" child="block7"/>
+  <xacro:voxel name="block8" origin="0 ${-1*cell_step} ${1.5*cell_step}" color="${blue}"/>
+  <xacro:joint_fix name="fixed7_8" parent="block7" child="block8"/>
+  <xacro:voxel name="block9_rev" origin="0 ${0*cell_step} ${-0.5*cell_step}" color="${green}"/>
+  <xacro:joint_revolution name="rev8_9" parent="block8" child="block9_rev" axis="0 1 0" origin="0 ${0*cell_step} ${2*cell_step}" rpy="1.57 0 0"/>
+  <xacro:voxel name="block10" origin="0 0 ${-0.5*cell_step}" color="${green}"/>
+  <xacro:joint_revolution name="rev9_10" parent="block9_rev" child="block10" axis="0 0 1" origin="0 0 ${1*cell_step}" rpy="0 0 0"/>
+  <xacro:voxel name="block14_fix" origin="0 0 ${0.5*cell_step}" color="${red}"/>
+  <xacro:joint_fix name="fixed13_14" parent="block10" child="block14_fix"/>
   <ros2_control name="GazeboSimSystem" type="system">
     <hardware>
@@ -80,5 +86,17 @@
       <state_interface name="position"/>
     </joint>
-    <joint name="rev4_5">
+    <joint name="rev2_3">
+      <command_interface name="position"/>
+      <state_interface name="position"/>
+    </joint>
+    <joint name="rev5_6">
+      <command_interface name="position"/>
+      <state_interface name="position"/>
+    </joint>
+    <joint name="rev8_9">
+      <command_interface name="position"/>
+      <state_interface name="position"/>
+    </joint>
+    <joint name="rev9_10">
       <command_interface name="position"/>
       <state_interface name="position"/>
@@ -89,4 +107,11 @@
       <parameters>$(find srrs_sim)/config/two_blocks_controller.yaml</parameters>
     </plugin>
+    <!--  CHECK THIS
+    <plugin name="gazebo_ros_state" filename="libgazebo_ros_state.so">
+      <ros>
+        <namespace>/gazebo</namespace>
+      </ros>
+    </plugin>
+    -->
   </gazebo>
 </robot>

Commit message: implemented simple going algorithm

File: ros2_ws/src/srrs_sim/urdf/robot.xacro (robot description, xacro)
@@ -53,7 +53,7 @@
     <xacro:joint_fix name="${name}visualfixed" parent="${parent}" child="${name}visual"/>
   </xacro:macro>
-  <link name="world"/>
+  <!-- <link name="world"/> -->
   <xacro:voxel name="block0_fix" origin="0 0 0" color="${red}"/>
-  <xacro:joint_fix name="world_to_base" parent="world" child="block0_fix"/>
+  <!-- <xacro:joint_fix name="world_to_base" parent="world" child="block0_fix"/> -->
   <xacro:voxel name="block1_rev" origin="0 0 0" color="${green}"/>
   <xacro:joint_revolution name="rev0_1" parent="block0_fix" child="block1_rev" axis="0 0 1" origin="0 0 ${cell_step}" rpy="0 0 0"/>
@@ -74,8 +74,8 @@
   <xacro:voxel name="block9_rev" origin="0 ${0*cell_step} ${-0.5*cell_step}" color="${green}"/>
   <xacro:joint_revolution name="rev8_9" parent="block8" child="block9_rev" axis="0 1 0" origin="0 ${0*cell_step} ${2*cell_step}" rpy="1.57 0 0"/>
-  <xacro:voxel name="block10" origin="0 0 ${-0.5*cell_step}" color="${green}"/>
-  <xacro:joint_revolution name="rev9_10" parent="block9_rev" child="block10" axis="0 0 1" origin="0 0 ${1*cell_step}" rpy="0 0 0"/>
-  <xacro:voxel name="block14_fix" origin="0 0 ${0.5*cell_step}" color="${red}"/>
-  <xacro:joint_fix name="fixed13_14" parent="block10" child="block14_fix"/>
+  <xacro:voxel name="block10" origin="0 0 ${0.5*cell_step}" color="${green}"/>
+  <xacro:joint_fix name="fixed9_10" parent="block9_rev" child="block10"/>
+  <xacro:voxel name="block14fix" origin="0 0 0" color="${red}"/>
+  <xacro:joint_revolution name="rev13_14" parent="block10" child="block14fix" axis="0 0 1" origin="0 0 ${1.5*cell_step}" rpy="0 0 0"/>
   <ros2_control name="GazeboSimSystem" type="system">
     <hardware>
@@ -98,5 +98,5 @@
       <state_interface name="position"/>
     </joint>
-    <joint name="rev9_10">
+    <joint name="rev13_14">
       <command_interface name="position"/>
       <state_interface name="position"/>
@@ -108,5 +108,5 @@
       <parameters>$(find srrs_sim)/config/robot_controller.yaml</parameters>
     </plugin>
-    <plugin
+    <!-- <plugin
       filename="libgz-sim8-detachable-joint-system.so"
       name="gz::sim::systems::DetachableJoint">
@@ -114,7 +114,27 @@
       <child_model>voxel</child_model>
       <child_link>voxel_link</child_link>
-      <attach_topic>attach_link</attach_topic>
-      <detach_topic>detach_link</detach_topic>
-      <output_topic>detachable_link_state</output_topic>
+      <attach_topic>attach_link_voxel</attach_topic>
+      <detach_topic>detach_link_voxel</detach_topic>
+      <output_topic>detachable_link_voxel_state</output_topic>
+    </plugin> -->
+    <plugin
+      filename="libgz-sim8-detachable-joint-system.so"
+      name="gz::sim::systems::DetachableJoint">
+      <parent_link>block0_fix</parent_link>
+      <child_model>box_base</child_model>
+      <child_link>base_link</child_link>
+      <attach_topic>attach_link1</attach_topic>
+      <detach_topic>detach_link1</detach_topic>
+      <output_topic>detachable_link_state1</output_topic>
+    </plugin>
+    <plugin
+      filename="libgz-sim8-detachable-joint-system.so"
+      name="gz::sim::systems::DetachableJoint">
+      <parent_link>block14fix</parent_link>
+      <child_model>box_base</child_model>
+      <child_link>base_link</child_link>
+      <attach_topic>attach_link2</attach_topic>
+      <detach_topic>detach_link2</detach_topic>
+      <output_topic>detachable_link_state2</output_topic>
     </plugin>
   </gazebo>

Commit message: Changing specifications and algorithms

File: ros2_ws/src/srrs_sim/urdf/robot.xacro (robot description, xacro)
@@ -78,4 +78,26 @@
   <xacro:voxel name="block14fix" origin="0 0 0" color="${red}"/>
   <xacro:joint_revolution name="rev13_14" parent="block10" child="block14fix" axis="0 0 1" origin="0 0 ${1.5*cell_step}" rpy="0 0 0"/>
+  <link name="camera_link">
+    <visual name="camera_link_visual">
+      <geometry>
+        <box size="0.05 0.05 0.05"/>
+      </geometry>
+    </visual>
+    <inertial>
+      <mass value="0.1"/>
+      <inertia ixx="0.0001" ixy="0.0" ixz="0.0" iyy="0.0001" iyz="0.0" izz="0.0001"/>
+    </inertial>
+  </link>
+  <joint name="camera_joint" type="fixed">
+    <parent link="block14fix"/>
+    <child link="camera_link"/>
+    <origin xyz="0.1 0 0" rpy="0 0 0"/>
+  </joint>
+  <link name="camera_link_optical"/>
+  <joint name="camera_optical_joint" type="fixed">
+    <parent link="camera_link"/>
+    <child link="camera_link_optical"/>
+    <origin xyz="0 0 0" rpy="-1.5708 0 -1.5708"/>
+  </joint>
   <ros2_control name="GazeboSimSystem" type="system">
     <hardware>
@@ -111,5 +133,5 @@
       filename="libgz-sim8-detachable-joint-system.so"
       name="gz::sim::systems::DetachableJoint">
-      <parent_link>block10</parent_link>
+      <parent_link>block14fix</parent_link>
       <child_model>voxel</child_model>
       <child_link>voxel_link</child_link>
@@ -122,5 +144,5 @@
       name="gz::sim::systems::DetachableJoint">
       <parent_link>block0_fix</parent_link>
-      <child_model>box_base</child_model>
+      <child_model>base</child_model>
       <child_link>base_link</child_link>
       <attach_topic>attach_link1</attach_topic>
@@ -132,5 +154,5 @@
       name="gz::sim::systems::DetachableJoint">
       <parent_link>block14fix</parent_link>
-      <child_model>box_base</child_model>
+      <child_model>base</child_model>
       <child_link>base_link</child_link>
       <attach_topic>attach_link2</attach_topic>
@@ -138,5 +160,24 @@
       <output_topic>detachable_link_state2</output_topic>
     </plugin>
+    <sensor name="camera_sensor" type="camera">
+      <always_on>1</always_on>
+      <update_rate>30.0</update_rate>
+      <camera>
+        <horizontal_fov>1.5708</horizontal_fov> <!-- 90 degrees in radians -->
+        <image>
+          <width>640</width>
+          <height>480</height>
+          <format>R8G8B8</format>
+        </image>
+        <clip>
+          <near>0.1</near>
+          <far>100</far>
+        </clip>
+      </camera>
+      <plugin name="camera_plugin" filename="libgz-sensors8-camera.so">
+        <topic_name>/camera/image_raw</topic_name>
+        <frame_name>camera_link</frame_name>
+      </plugin>
+    </sensor>
   </gazebo>
-  <!-- ros2 run ros_gz_bridge parameter_bridge   /attach_link@std_msgs/msg/Empty@gz.msgs.Empty   /detach_link@std_msgs/msg/Empty@gz.msgs.Empty -->
 </robot>

Commit message: add gui, collision to part and base

File: ros2_ws/src/srrs_sim/urdf/robot.xacro (robot description, xacro)
@@ -10,7 +10,14 @@
         <geometry>
             <mesh filename="/home/lao/Documents/Masterarbeit/git/SRRS_gazebo_sim/ros2_ws/src/srrs_sim/meshes/Voxel.stl" scale="0.001 0.001 0.001"/>
+            <!-- <box size="0.1 0.1 0.1"/> -->
         </geometry>
         <origin xyz="${origin}"/>
       </visual>
+      <collision>
+         <geometry>
+          <mesh filename="/home/lao/Documents/Masterarbeit/git/SRRS_gazebo_sim/ros2_ws/src/srrs_sim/meshes/Voxel.stl" scale="0.001 0.001 0.001"/>
+            <!-- <box size="0.1 0.1 0.1"/> -->
+         </geometry>
+      </collision>
       <inertial>
         <mass value="0.1"/>

Commit message: updated goto_xyz to any possible XYZ

File: ros2_ws/src/srrs_sim/urdf/robot.xacro (robot description, xacro)
@@ -4,4 +4,6 @@
   <xacro:property name="red" value="0.8 0 0 1" />
   <xacro:property name="blue" value="0 0 0.8 1" />
+  <xacro:property name="yellow" value="1 1 0 1" />
+  <xacro:property name="white" value="1 1 1 1" />
   <xacro:property name="cell_step" value="0.134"/>
   <xacro:macro name="voxel" params="name origin color" >
@@ -83,5 +85,5 @@
   <xacro:voxel name="block10" origin="0 0 ${0.5*cell_step}" color="${green}"/>
   <xacro:joint_fix name="fixed9_10" parent="block9_rev" child="block10"/>
-  <xacro:voxel name="block14fix" origin="0 0 0" color="${red}"/>
+  <xacro:voxel name="block14fix" origin="0 0 0" color="${yellow}"/>
   <xacro:joint_revolution name="rev13_14" parent="block10" child="block14fix" axis="0 0 1" origin="0 0 ${1.5*cell_step}" rpy="0 0 0"/>
   <link name="camera_link">
@@ -95,4 +97,22 @@
       <inertia ixx="0.0001" ixy="0.0" ixz="0.0" iyy="0.0001" iyz="0.0" izz="0.0001"/>
     </inertial>
+    <sensor name="camera_sensor" type="camera">
+      <always_on>1</always_on>
+      <update_rate>30.0</update_rate>
+      <visualize>true</visualize>
+      <topic>/camera/image_raw</topic>
+      <camera>
+        <horizontal_fov>1.5708</horizontal_fov> <!-- 90 degrees in radians -->
+        <image>
+          <width>640</width>
+          <height>480</height>
+          <format>R8G8B8</format>
+        </image>
+        <clip>
+          <near>0.1</near>
+          <far>100</far>
+        </clip>
+      </camera>
+    </sensor>
   </link>
   <joint name="camera_joint" type="fixed">
@@ -137,14 +157,4 @@
       <parameters>$(find srrs_sim)/config/robot_controller.yaml</parameters>
     </plugin>
-    <!-- <plugin
-      filename="libgz-sim8-detachable-joint-system.so"
-      name="gz::sim::systems::DetachableJoint">
-      <parent_link>block14fix</parent_link>
-      <child_model>voxel</child_model>
-      <child_link>voxel_link</child_link>
-      <attach_topic>attach_link_voxel</attach_topic>
-      <detach_topic>detach_link_voxel</detach_topic>
-      <output_topic>detachable_link_voxel_state</output_topic>
-    </plugin> -->
     <plugin
       filename="libgz-sim8-detachable-joint-system.so"
@@ -187,24 +197,8 @@
       <output_topic>detachable_obj_link_state2</output_topic>
     </plugin>
-    <sensor name="camera_sensor" type="camera">
-      <always_on>1</always_on>
-      <update_rate>30.0</update_rate>
-      <camera>
-        <horizontal_fov>1.5708</horizontal_fov> <!-- 90 degrees in radians -->
-        <image>
-          <width>640</width>
-          <height>480</height>
-          <format>R8G8B8</format>
-        </image>
-        <clip>
-          <near>0.1</near>
-          <far>100</far>
-        </clip>
-      </camera>
-      <plugin name="camera_plugin" filename="libgz-sensors8-camera.so">
-        <topic_name>/camera/image_raw</topic_name>
-        <frame_name>camera_link</frame_name>
-      </plugin>
-    </sensor>
+    <!-- <plugin name="gz::sim::systems::LogicalCamera" filename="libgz-sim8-logical-camera-system.so">
+      <topic_name>/camera/image_raw</topic_name>
+      <frame_name>camera_link</frame_name>
+    </plugin> -->
   </gazebo>
 </robot>

Commit message: fix lack of sensors in gz, through adding sensors plugin in world.sdf, added camera sensor in head_camera.sdf, not fixed to robot

File: ros2_ws/src/srrs_sim/urdf/robot.xacro (robot description, xacro)
@@ -97,34 +97,15 @@
       <inertia ixx="0.0001" ixy="0.0" ixz="0.0" iyy="0.0001" iyz="0.0" izz="0.0001"/>
     </inertial>
-    <sensor name="camera_sensor" type="camera">
-      <always_on>1</always_on>
-      <update_rate>30.0</update_rate>
-      <visualize>true</visualize>
-      <topic>/camera/image_raw</topic>
-      <camera>
-        <horizontal_fov>1.5708</horizontal_fov> <!-- 90 degrees in radians -->
-        <image>
-          <width>640</width>
-          <height>480</height>
-          <format>R8G8B8</format>
-        </image>
-        <clip>
-          <near>0.1</near>
-          <far>100</far>
-        </clip>
-      </camera>
-    </sensor>
   </link>
-  <joint name="camera_joint" type="fixed">
+  <joint name="camera_visual_block_joint" type="fixed">
     <parent link="block14fix"/>
     <child link="camera_link"/>
     <origin xyz="0.1 0 0" rpy="0 0 0"/>
   </joint>
-  <link name="camera_link_optical"/>
-  <joint name="camera_optical_joint" type="fixed">
+  <!-- <joint name="camera_joint" type="fixed">
     <parent link="camera_link"/>
-    <child link="camera_link_optical"/>
-    <origin xyz="0 0 0" rpy="-1.5708 0 -1.5708"/>
-  </joint>
+    <child link="sensor_link"/>
+    <origin xyz="0.1 0 0" rpy="0 0 0"/>
+  </joint> -->
   <ros2_control name="GazeboSimSystem" type="system">
     <hardware>
@@ -197,8 +178,4 @@
       <output_topic>detachable_obj_link_state2</output_topic>
     </plugin>
-    <!-- <plugin name="gz::sim::systems::LogicalCamera" filename="libgz-sim8-logical-camera-system.so">
-      <topic_name>/camera/image_raw</topic_name>
-      <frame_name>camera_link</frame_name>
-    </plugin> -->
   </gazebo>
 </robot>

Commit message: fix camera to robot, tried to add contact sensor but doent work, launch file error with controller timeout

File: ros2_ws/src/srrs_sim/urdf/robot.xacro (robot description, xacro)
@@ -16,5 +16,5 @@
         <origin xyz="${origin}"/>
       </visual>
-      <collision>
+      <collision name="${name}_collision">
          <geometry>
           <mesh filename="/home/lao/Documents/Masterarbeit/git/SRRS_gazebo_sim/ros2_ws/src/srrs_sim/meshes/Voxel.stl" scale="0.001 0.001 0.001"/>
@@ -61,4 +61,24 @@
     </link>
     <xacro:joint_fix name="${name}visualfixed" parent="${parent}" child="${name}visual"/>
+  </xacro:macro>
+  <xacro:macro name="contact_plate" params="name parent" >
+    <link name="${name}">
+      <visual>
+        <geometry>
+            <box size="0.1 0.1 0.01"/>
+        </geometry>
+        <!-- <origin xyz="${origin}"/> -->
+      </visual>
+      <collision name="${name}_collision">
+        <geometry>
+          <box size="0.1 0.1 0.01"/>
+        </geometry>
+      </collision>
+    </link>
+    <joint name="${name}_joint" type="fixed">
+      <origin xyz="0 0 0.2"/>
+      <parent link="${parent}"/>
+      <child link="${name}"/>
+    </joint>
   </xacro:macro>
   <!-- <link name="world"/> -->
@@ -87,4 +107,5 @@
   <xacro:voxel name="block14fix" origin="0 0 0" color="${yellow}"/>
   <xacro:joint_revolution name="rev13_14" parent="block10" child="block14fix" axis="0 0 1" origin="0 0 ${1.5*cell_step}" rpy="0 0 0"/>
+  <!-- <xacro:contact_plate name="block14fix_contact" parent="block14fix"/> -->
   <link name="camera_link">
     <visual name="camera_link_visual">
@@ -178,4 +199,40 @@
       <output_topic>detachable_obj_link_state2</output_topic>
     </plugin>
+    <plugin
+      filename="gz-sim-contact-system"
+      name="gz::sim::systems::Contact"/>
+  </gazebo>
+  <gazebo reference="camera_link">
+    <sensor name="camera_sensor" type="camera">
+      <camera>
+        <horizontal_fov>1.3962634</horizontal_fov>
+        <image>
+          <width>640</width>
+          <height>480</height>
+          <format>R8G8B8</format>
+        </image>
+        <clip>
+          <near>0.1</near>
+          <far>15</far>
+        </clip>
+        <optical_frame_id>camera_link_optical</optical_frame_id>
+        <camera_info_topic>camera/camera_info</camera_info_topic>
+      </camera>
+      <always_on>1</always_on>
+      <update_rate>20</update_rate>
+      <visualize>true</visualize>
+      <topic>camera/image</topic>
+    </sensor>
+  </gazebo>
+  <gazebo reference="block14fix_contact">
+    <sensor name="contact_sensor" type="contact">
+      <contact>
+        <!-- Match the collision element name in the link -->
+        <collision>block14fix_contact_collision</collision>
+      </contact>
+      <always_on>true</always_on>
+      <update_rate>100</update_rate>
+      <topic>robot/contacts</topic>
+    </sensor>
   </gazebo>
 </robot>
