Commit message: fixed joint_position_controllers bugs, fixed camera by adding _optical link frame

File: ros2_ws/src/srrs_sim/urdf/robot.xacro (robot description, xacro)
@@ -114,93 +114,15 @@
       </geometry>
     </visual>
-    <inertial>
-      <mass value="0.1"/>
-      <inertia ixx="0.0001" ixy="0.0" ixz="0.0" iyy="0.0001" iyz="0.0" izz="0.0001"/>
-    </inertial>
   </link>
-  <joint name="camera_visual_block_joint" type="fixed">
+  <joint name="camera_joint" type="fixed">
     <parent link="block14fix"/>
     <child link="camera_link"/>
-    <origin xyz="0.1 0 0" rpy="0 0 0"/>
   </joint>
-  <!-- <joint name="camera_joint" type="fixed">
+  <link name="camera_link_optical"></link>
+  <joint name="camera_optical_joint" type="fixed">
     <parent link="camera_link"/>
-    <child link="sensor_link"/>
-    <origin xyz="0.1 0 0" rpy="0 0 0"/>
-  </joint> -->
-  <ros2_control name="GazeboSimSystem" type="system">
-    <hardware>
-      <plugin>gz_ros2_control/GazeboSimSystem</plugin>
-    </hardware>
-    <joint name="rev0_1">
-      <command_interface name="position"/>
-      <state_interface name="position"/>
-    </joint>
-    <joint name="rev2_3">
-      <command_interface name="position"/>
-      <state_interface name="position"/>
-    </joint>
-    <joint name="rev5_6">
-      <command_interface name="position"/>
-      <state_interface name="position"/>
-    </joint>
-    <joint name="rev8_9">
-      <command_interface name="position"/>
-      <state_interface name="position"/>
-    </joint>
-    <joint name="rev13_14">
-      <command_interface name="position"/>
-      <state_interface name="position"/>
-    </joint>
-  </ros2_control>
-  <gazebo>
-    <plugin filename="gz_ros2_control-system" name="gz_ros2_control::GazeboSimROS2ControlPlugin">
-      <!-- <parameters>$(find srrs_sim)/config/two_blocks_controller.yaml</parameters> -->
-      <parameters>$(find srrs_sim)/config/robot_controller.yaml</parameters>
-    </plugin>
-    <plugin
-      filename="libgz-sim8-detachable-joint-system.so"
-      name="gz::sim::systems::DetachableJoint">
-      <parent_link>block0_fix</parent_link>
-      <child_model>base</child_model>
-      <child_link>base_link</child_link>
-      <attach_topic>attach_link1</attach_topic>
-      <detach_topic>detach_link1</detach_topic>
-      <output_topic>detachable_link_state1</output_topic>
-    </plugin>
-    <plugin
-      filename="libgz-sim8-detachable-joint-system.so"
-      name="gz::sim::systems::DetachableJoint">
-      <parent_link>block14fix</parent_link>
-      <child_model>base</child_model>
-      <child_link>base_link</child_link>
-      <attach_topic>attach_link2</attach_topic>
-      <detach_topic>detach_link2</detach_topic>
-      <output_topic>detachable_link_state2</output_topic>
-    </plugin>
-    <plugin
-      filename="libgz-sim8-detachable-joint-system.so"
-      name="gz::sim::systems::DetachableJoint">
-      <parent_link>block0_fix</parent_link>
-      <child_model>voxel</child_model>
-      <child_link>voxel</child_link>
-      <attach_topic>attach_obj_link1</attach_topic>
-      <detach_topic>detach_obj_link1</detach_topic>
-      <output_topic>detachable_obj_link_state1</output_topic>
-    </plugin>
-    <plugin
-      filename="libgz-sim8-detachable-joint-system.so"
-      name="gz::sim::systems::DetachableJoint">
-      <parent_link>block14fix</parent_link>
-      <child_model>voxel</child_model>
-      <child_link>voxel</child_link>
-      <attach_topic>attach_obj_link2</attach_topic>
-      <detach_topic>detach_obj_link2</detach_topic>
-      <output_topic>detachable_obj_link_state2</output_topic>
-    </plugin>
-    <plugin
-      filename="gz-sim-contact-system"
-      name="gz::sim::systems::Contact"/>
-  </gazebo>
+    <child link="camera_link_optical"/>
+    <origin xyz = "0 0 0" rpy = "${-pi/2} 0 ${-pi/2}"/>
+  </joint>
   <gazebo reference="camera_link">
     <sensor name="camera_sensor" type="camera">
@@ -225,4 +147,78 @@
     </sensor>
   </gazebo>
+  <ros2_control name="GazeboSimSystem" type="system">
+    <hardware>
+      <plugin>gz_ros2_control/GazeboSimSystem</plugin>
+    </hardware>
+    <joint name="rev0_1">
+      <command_interface name="position"/>
+      <state_interface name="position"/>
+    </joint>
+    <joint name="rev2_3">
+      <command_interface name="position"/>
+      <state_interface name="position"/>
+    </joint>
+    <joint name="rev5_6">
+      <command_interface name="position"/>
+      <state_interface name="position"/>
+    </joint>
+    <joint name="rev8_9">
+      <command_interface name="position"/>
+      <state_interface name="position"/>
+    </joint>
+    <joint name="rev13_14">
+      <command_interface name="position"/>
+      <state_interface name="position"/>
+    </joint>
+  </ros2_control>
+  <gazebo>
+    <plugin filename="gz_ros2_control-system" name="gz_ros2_control::GazeboSimROS2ControlPlugin">
+      <!-- <parameters>$(find srrs_sim)/config/two_blocks_controller.yaml</parameters> -->
+      <parameters>$(find srrs_sim)/config/robot_controller.yaml</parameters>
+    </plugin>
+    <plugin
+      filename="libgz-sim8-detachable-joint-system.so"
+      name="gz::sim::systems::DetachableJoint">
+      <parent_link>block0_fix</parent_link>
+      <child_model>base</child_model>
+      <child_link>base_link</child_link>
+      <attach_topic>attach_link1</attach_topic>
+      <detach_topic>detach_link1</detach_topic>
+      <output_topic>detachable_link_state1</output_topic>
+    </plugin>
+    <plugin
+      filename="libgz-sim8-detachable-joint-system.so"
+      name="gz::sim::systems::DetachableJoint">
+      <parent_link>block14fix</parent_link>
+      <child_model>base</child_model>
+      <child_link>base_link</child_link>
+      <attach_topic>attach_link2</attach_topic>
+      <detach_topic>detach_link2</detach_topic>
+      <output_topic>detachable_link_state2</output_topic>
+    </plugin>
+    <plugin
+      filename="libgz-sim8-detachable-joint-system.so"
+      name="gz::sim::systems::DetachableJoint">
+      <parent_link>block0_fix</parent_link>
+      <child_model>voxel</child_model>
+      <child_link>voxel</child_link>
+      <attach_topic>attach_obj_link1</attach_topic>
+      <detach_topic>detach_obj_link1</detach_topic>
+      <output_topic>detachable_obj_link_state1</output_topic>
+    </plugin>
+    <plugin
+      filename="libgz-sim8-detachable-joint-system.so"
+      name="gz::sim::systems::DetachableJoint">
+      <parent_link>block14fix</parent_link>
+      <child_model>voxel</child_model>
+      <child_link>voxel</child_link>
+      <attach_topic>attach_obj_link2</attach_topic>
+      <detach_topic>detach_obj_link2</detach_topic>
+      <output_topic>detachable_obj_link_state2</output_topic>
+    </plugin>
+    <plugin
+      filename="gz-sim-contact-system"
+      name="gz::sim::systems::Contact"/>
+  </gazebo>
   <gazebo reference="block14fix_contact">
     <sensor name="contact_sensor" type="contact">

Commit message: fixed contact sensor

File: ros2_ws/src/srrs_sim/urdf/robot.xacro (robot description, xacro)
@@ -7,4 +7,5 @@
   <xacro:property name="white" value="1 1 1 1" />
   <xacro:property name="cell_step" value="0.134"/>
+<!-- MACROS -->
   <xacro:macro name="voxel" params="name origin color" >
     <link name="${name}">
@@ -82,7 +83,6 @@
     </joint>
   </xacro:macro>
-  <!-- <link name="world"/> -->
+<!-- MAIN STRUCTURE -->
   <xacro:voxel name="block0_fix" origin="0 0 0" color="${red}"/>
-  <!-- <xacro:joint_fix name="world_to_base" parent="world" child="block0_fix"/> -->
   <xacro:voxel name="block1_rev" origin="0 0 0" color="${green}"/>
   <xacro:joint_revolution name="rev0_1" parent="block0_fix" child="block1_rev" axis="0 0 1" origin="0 0 ${cell_step}" rpy="0 0 0"/>
@@ -107,5 +107,5 @@
   <xacro:voxel name="block14fix" origin="0 0 0" color="${yellow}"/>
   <xacro:joint_revolution name="rev13_14" parent="block10" child="block14fix" axis="0 0 1" origin="0 0 ${1.5*cell_step}" rpy="0 0 0"/>
-  <!-- <xacro:contact_plate name="block14fix_contact" parent="block14fix"/> -->
+  <!-- CAMERA PART -->
   <link name="camera_link">
     <visual name="camera_link_visual">
@@ -127,4 +127,5 @@
   <gazebo reference="camera_link">
     <sensor name="camera_sensor" type="camera">
+    <visualize>true</visualize>
       <camera>
         <horizontal_fov>1.3962634</horizontal_fov>
@@ -147,4 +148,36 @@
     </sensor>
   </gazebo>
+  <!--  CONTACT SENSOR -->
+   <!-- <xacro:contact_plate name="block14fix_contact" parent="block14fix"/> -->
+  <link name="contact_link">
+    <visual>
+      <geometry>
+          <box size="0.1 0.1 0.001"/>
+      </geometry>
+      <!-- <origin xyz="${origin}"/> -->
+    </visual>
+    <collision name="contact_link_collision">
+      <geometry>
+        <box size="0.1 0.1 0.001"/>
+      </geometry>
+    </collision>
+  </link>
+  <joint name="contact_link_joint" type="fixed">
+    <origin xyz="0 0 0.137"/>
+    <parent link="block14fix"/>
+    <child link="contact_link"/>
+  </joint>
+  <gazebo reference="contact_link">
+    <sensor name="contact_sensor" type="contact">
+      <contact>
+      <!-- If doesnt work - check contact collision name in SDF, transfer xacro to urdf to sdf -->
+        <collision>block14fix_fixed_joint_lump__contact_link_collision_collision_1</collision>
+        <topic>/robot/contact2</topic>
+      </contact>
+      <always_on>true</always_on>
+      <update_rate>50</update_rate>
+    </sensor>
+  </gazebo>
+<!-- JOINTS CONTROL -->
   <ros2_control name="GazeboSimSystem" type="system">
     <hardware>
@@ -219,16 +252,6 @@
     <plugin
       filename="gz-sim-contact-system"
-      name="gz::sim::systems::Contact"/>
-  </gazebo>
-  <gazebo reference="block14fix_contact">
-    <sensor name="contact_sensor" type="contact">
-      <contact>
-        <!-- Match the collision element name in the link -->
-        <collision>block14fix_contact_collision</collision>
-      </contact>
-      <always_on>true</always_on>
-      <update_rate>100</update_rate>
-      <topic>robot/contacts</topic>
-    </sensor>
+      name="gz::sim::systems::Contact">
+    </plugin>
   </gazebo>
 </robot>

Commit message: xacro macro for contact sensor

File: ros2_ws/src/srrs_sim/urdf/robot.xacro (robot description, xacro)
@@ -63,9 +63,9 @@
     <xacro:joint_fix name="${name}visualfixed" parent="${parent}" child="${name}visual"/>
   </xacro:macro>
-  <xacro:macro name="contact_plate" params="name parent" >
+  <xacro:macro name="contact_plate" params="name parent origin" >
     <link name="${name}">
       <visual>
         <geometry>
-            <box size="0.1 0.1 0.01"/>
+            <cylinder radius="0.03" length="0.001"/>
         </geometry>
         <!-- <origin xyz="${origin}"/> -->
@@ -73,13 +73,24 @@
       <collision name="${name}_collision">
         <geometry>
-          <box size="0.1 0.1 0.01"/>
+          <cylinder radius="0.03" length="0.001"/>
         </geometry>
       </collision>
     </link>
     <joint name="${name}_joint" type="fixed">
-      <origin xyz="0 0 0.2"/>
+      <origin xyz="${origin}"/>
       <parent link="${parent}"/>
       <child link="${name}"/>
     </joint>
+    <gazebo reference="${name}">
+      <sensor name="${name}_sensor" type="contact">
+        <contact>
+        <!-- If doesnt work - check contact collision name in SDF, transfer xacro to urdf to sdf -->
+          <collision>${parent}_fixed_joint_lump__${name}_collision_collision_1</collision>
+          <topic>/robot/${name}</topic>
+        </contact>
+        <always_on>true</always_on>
+        <update_rate>50</update_rate>
+      </sensor>
+    </gazebo>
   </xacro:macro>
 <!-- MAIN STRUCTURE -->
@@ -148,35 +159,7 @@
     </sensor>
   </gazebo>
-  <!--  CONTACT SENSOR -->
-   <!-- <xacro:contact_plate name="block14fix_contact" parent="block14fix"/> -->
-  <link name="contact_link">
-    <visual>
-      <geometry>
-          <box size="0.1 0.1 0.001"/>
-      </geometry>
-      <!-- <origin xyz="${origin}"/> -->
-    </visual>
-    <collision name="contact_link_collision">
-      <geometry>
-        <box size="0.1 0.1 0.001"/>
-      </geometry>
-    </collision>
-  </link>
-  <joint name="contact_link_joint" type="fixed">
-    <origin xyz="0 0 0.137"/>
-    <parent link="block14fix"/>
-    <child link="contact_link"/>
-  </joint>
-  <gazebo reference="contact_link">
-    <sensor name="contact_sensor" type="contact">
-      <contact>
-      <!-- If doesnt work - check contact collision name in SDF, transfer xacro to urdf to sdf -->
-        <collision>block14fix_fixed_joint_lump__contact_link_collision_collision_1</collision>
-        <topic>/robot/contact2</topic>
-      </contact>
-      <always_on>true</always_on>
-      <update_rate>50</update_rate>
-    </sensor>
-  </gazebo>
+  <!--  CONTACT sensors -->
+   <xacro:contact_plate name="contact1" parent="block0_fix" origin="0 0 0"/>
+   <xacro:contact_plate name="contact2" parent="block14fix" origin="0 0 0.137"/>
 <!-- JOINTS CONTROL -->
   <ros2_control name="GazeboSimSystem" type="system">

File: ros2_ws/src/srrs_sim/urdf/temp_robot.urdf (robot description, URDF)
Before this commit: robot rel_robot, 20 links, 19 joints
Links:
- removed link contact_link
- added link contact1; collision cylinder length=0.001 radius=0.07; visual cylinder length=0.001 radius=0.07
- added link contact2; collision cylinder length=0.001 radius=0.07; visual cylinder length=0.001 radius=0.07
Joints:
- removed joint contact_link_joint
- added joint contact1_joint: type fixed, parent block0_fix, child contact1, origin xyz=0 0 0
- added joint contact2_joint: type fixed, parent block14fix, child contact2, origin xyz=0 0 0.137

Commit message: added camera xacro, need to fix rpy rotation angles of camera

File: ros2_ws/src/srrs_sim/urdf/robot.xacro (robot description, xacro)
@@ -91,4 +91,46 @@
         <always_on>true</always_on>
         <update_rate>50</update_rate>
+      </sensor>
+    </gazebo>
+  </xacro:macro>
+  <xacro:macro name="camera_sensor" params="name parent origin_xyz origin_rpy" >
+    <link name="${name}">
+      <visual name="${name}_visual">
+        <geometry>
+          <box size="0.05 0.05 0.05"/>
+        </geometry>
+      </visual>
+    </link>
+    <joint name="${name}_joint" type="fixed">
+      <parent link="${parent}"/>
+      <child link="${name}"/>
+    </joint>
+    <link name="${name}_optical"></link>
+    <joint name="${name}_optical_joint" type="fixed">
+      <parent link="${name}"/>
+      <child link="${name}_optical"/>
+      <origin xyz="${origin_xyz}" rpy="${origin_rpy}"/>
+    </joint>
+    <gazebo reference="${name}">
+      <sensor name="${name}_sensor" type="camera">
+      <visualize>true</visualize>
+        <camera>
+          <horizontal_fov>1.3962634</horizontal_fov>
+          <image>
+            <width>640</width>
+            <height>480</height>
+            <format>R8G8B8</format>
+          </image>
+          <clip>
+            <near>0.1</near>
+            <far>15</far>
+          </clip>
+          <optical_frame_id>${name}_optical</optical_frame_id>
+          <camera_info_topic>/${name}/camera_info</camera_info_topic>
+        </camera>
+        <always_on>1</always_on>
+        <update_rate>20</update_rate>
+        <visualize>true</visualize>
+        <topic>/${name}/image</topic>
       </sensor>
     </gazebo>
@@ -119,44 +161,6 @@
   <xacro:joint_revolution name="rev13_14" parent="block10" child="block14fix" axis="0 0 1" origin="0 0 ${1.5*cell_step}" rpy="0 0 0"/>
   <!-- CAMERA PART -->
-  <link name="camera_link">
-    <visual name="camera_link_visual">
-      <geometry>
-        <box size="0.05 0.05 0.05"/>
-      </geometry>
-    </visual>
-  </link>
-  <joint name="camera_joint" type="fixed">
-    <parent link="block14fix"/>
-    <child link="camera_link"/>
-  </joint>
-  <link name="camera_link_optical"></link>
-  <joint name="camera_optical_joint" type="fixed">
-    <parent link="camera_link"/>
-    <child link="camera_link_optical"/>
-    <origin xyz = "0 0 0" rpy = "${-pi/2} 0 ${-pi/2}"/>
-  </joint>
-  <gazebo reference="camera_link">
-    <sensor name="camera_sensor" type="camera">
-    <visualize>true</visualize>
-      <camera>
-        <horizontal_fov>1.3962634</horizontal_fov>
-        <image>
-          <width>640</width>
-          <height>480</height>
-          <format>R8G8B8</format>
-        </image>
-        <clip>
-          <near>0.1</near>
-          <far>15</far>
-        </clip>
-        <optical_frame_id>camera_link_optical</optical_frame_id>
-        <camera_info_topic>camera/camera_info</camera_info_topic>
-      </camera>
-      <always_on>1</always_on>
-      <update_rate>20</update_rate>
-      <visualize>true</visualize>
-      <topic>camera/image</topic>
-    </sensor>
-  </gazebo>
+  <xacro:camera_sensor name="camera1" parent="block0_fix" origin_xyz="0 0 0" origin_rpy="${-pi/2} ${-pi/2} ${-pi/2}"/>
+  <xacro:camera_sensor name="camera2" parent="block14fix" origin_xyz="0 0 0" origin_rpy="0 ${-pi/2} 0"/>
   <!--  CONTACT sensors -->
    <xacro:contact_plate name="contact1" parent="block0_fix" origin="0 0 0"/>

Commit message: separated sensor class node, logic to wait for contact during step - not finished

File: ros2_ws/src/srrs_sim/urdf/robot.xacro (robot description, xacro)
@@ -98,5 +98,5 @@
       <visual name="${name}_visual">
         <geometry>
-          <box size="0.05 0.05 0.05"/>
+          <box size="0.01 0.01 0.01"/>
         </geometry>
       </visual>
@@ -105,4 +105,5 @@
       <parent link="${parent}"/>
       <child link="${name}"/>
+      <origin xyz="${origin_xyz}" rpy="${origin_rpy}"/>
     </joint>
     <link name="${name}_optical"></link>
@@ -110,5 +111,5 @@
       <parent link="${name}"/>
       <child link="${name}_optical"/>
-      <origin xyz="${origin_xyz}" rpy="${origin_rpy}"/>
+      <origin xyz="0 0 0" rpy="${-pi/2} 0 ${-pi/2}"/>
     </joint>
     <gazebo reference="${name}">
@@ -161,6 +162,6 @@
   <xacro:joint_revolution name="rev13_14" parent="block10" child="block14fix" axis="0 0 1" origin="0 0 ${1.5*cell_step}" rpy="0 0 0"/>
   <!-- CAMERA PART -->
-  <xacro:camera_sensor name="camera1" parent="block0_fix" origin_xyz="0 0 0" origin_rpy="${-pi/2} ${-pi/2} ${-pi/2}"/>
-  <xacro:camera_sensor name="camera2" parent="block14fix" origin_xyz="0 0 0" origin_rpy="0 ${-pi/2} 0"/>
+  <xacro:camera_sensor name="camera1" parent="block0_fix" origin_xyz="0 0 0" origin_rpy="0 ${pi/2} 0"/>
+  <xacro:camera_sensor name="camera2" parent="block14fix" origin_xyz="0 0 ${1*cell_step}" origin_rpy="0 ${-pi/2} 0"/>
   <!--  CONTACT sensors -->
    <xacro:contact_plate name="contact1" parent="block0_fix" origin="0 0 0"/>

Commit message: joints angle feedback waiting cycle finished

File: ros2_ws/src/srrs_sim/urdf/robot.xacro (robot description, xacro)
@@ -67,5 +67,5 @@
       <visual>
         <geometry>
-            <cylinder radius="0.03" length="0.001"/>
+            <cylinder radius="0.05" length="0.002"/>
         </geometry>
         <!-- <origin xyz="${origin}"/> -->
@@ -73,5 +73,5 @@
       <collision name="${name}_collision">
         <geometry>
-          <cylinder radius="0.03" length="0.001"/>
+          <cylinder radius="0.05" length="0.002"/>
         </geometry>
       </collision>
@@ -134,4 +134,14 @@
         <visualize>true</visualize>
         <topic>/${name}/image</topic>
+      </sensor>
+    </gazebo>
+  </xacro:macro>
+  <xacro:macro name="imu_sensor" params="name parent">
+    <gazebo reference="${parent}">
+      <sensor name="imu_sensor" type="imu">
+          <always_on>1</always_on>
+          <update_rate>50</update_rate>
+          <visualize>true</visualize>
+          <topic>/robot/${name}</topic>
       </sensor>
     </gazebo>
@@ -166,5 +176,8 @@
   <!--  CONTACT sensors -->
    <xacro:contact_plate name="contact1" parent="block0_fix" origin="0 0 0"/>
-   <xacro:contact_plate name="contact2" parent="block14fix" origin="0 0 0.137"/>
+   <xacro:contact_plate name="contact2" parent="block14fix" origin="0 0 ${1*cell_step}"/>
+<!-- IMU sensors -->
+    <xacro:imu_sensor name="imu1" parent="block0_fix"/>
+    <xacro:imu_sensor name="imu2" parent="block14fix"/>
 <!-- JOINTS CONTROL -->
   <ros2_control name="GazeboSimSystem" type="system">
